File: zmpt101b - 3phase din.brd (EAGLE design)
At the start: 50 x 86.5 mm, 3 parts

Commit message: 1st version
Parts:
- added D1, D2, D3: DIODE_DO-219-AB(SOD123F), Diode:SODFL3718X115
- added R1, R10, R11, R12, R2, R3, R4, R5, R6, R7, R8, R9: (no value), rcl:R1206
- added U$1, U$2: 5MMBLOCK_X9, 5mm terminal block:9/5.08
- moved TR1 36.8 mm to (4.11, 28.5), turned to 0 degrees
- moved TR2 28.3 mm to (32.4, 71.8), flipped to the bottom, turned to 270 degrees
- moved TR3 24.8 mm to (26.0, 28.4), turned to 0 degrees
Connections:
- new net N$1: R3.1, U$1.P$1
- new net N$10: R5.2, TR2.P$4
- new net N$11: R8.2, TR2.P$3
- new net N$12: U$1.P$2
- new net N$13: R11.1, U$1.P$5
- new net N$14: R10.1, R11.2
- new net N$15: R10.2, R9.1
- new net N$16: R9.2, TR3.P$4
- new net N$17: R12.2, TR3.P$3
- new net N$18: U$1.P$4
- new net N$19: U$1.P$6
- new net N$2: R2.1, R3.2
- new net N$20: U$1.P$7
- new net N$21: U$1.P$8
- new net N$22: D1.1, TR1.P$1, U$2.P$9
- new net N$23: D1.2, TR1.P$2, U$2.P$8
- new net N$24: D2.1, TR2.P$1, U$2.P$6
- new net N$25: D2.2, TR2.P$2, U$2.P$5
- new net N$26: D3.1, TR3.P$1, U$2.P$3
- new net N$27: D3.2, TR3.P$2, U$2.P$2
- new net N$3: R1.1, R2.2
- new net N$4: R1.2, TR1.P$4
- new net N$5: R4.2, TR1.P$3
- new net N$6: R12.1, R4.1, R8.1, U$1.P$9
- new net N$7: R7.1, U$1.P$3
- new net N$8: R6.1, R7.2
- new net N$9: R5.1, R6.2
- new net P$1: U$2.P$1
- new net P$4: U$2.P$4
- new net P$7: U$2.P$7
Routing:
- net N$5: track 0.00 -> 66.7 mm, vias 0 -> 1
- net N$24: track 0.00 -> 57.0 mm
- net N$25: track 0.00 -> 55.7 mm
- net N$22: track 0.00 -> 44.8 mm
- net N$26: track 0.00 -> 41.2 mm
- net N$17: track 0.00 -> 38.2 mm, vias 0 -> 1
- net N$23: track 0.00 -> 31.0 mm
- net N$27: track 0.00 -> 26.8 mm
- net N$4: track 0.00 -> 21.6 mm
- net N$11: track 0.00 -> 21.1 mm, vias 0 -> 1
- net N$16: track 0.00 -> 20.7 mm
- net N$6: track 0.00 -> 19.7 mm
- net N$13: track 0.00 -> 13.8 mm
- net N$10: track 0.00 -> 8.08 mm
- net N$7: track 0.00 -> 7.21 mm
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Other:
- outline, holes or cut-outs redrawn

Commit message: commit v0.1 for prototyping
Parts:
- R1, R11, R12, R2, R3, R4, R5, R6, R7, R8, R9: value (none) -> 51k
- R10: value (none) -> 15k
- moved TR2 16.6 mm to (15.8, 71.7), flipped to the top
- moved R5 4.40 mm to (11.3, 59.9)
- moved R2 4.40 mm to (4.52, 65.6)
- moved R3 4.40 mm to (4.52, 71.1)
- moved R6 4.40 mm to (11.3, 65.4)
- moved R7 4.40 mm to (11.3, 70.9)
- moved R1 4.40 mm to (4.52, 60.1)
- moved R10 4.32 mm to (35.8, 64.4)
- moved R11 4.32 mm to (35.8, 70.5)
- moved R9 4.32 mm to (35.8, 58.1)
Connections:
- net P$1 renamed GND
- net N$10: now also R8.2; no longer R5.2
- net N$11: now also R5.2; no longer R8.2
- net N$24: now also TR2.P$2; no longer TR2.P$1
- net N$25: now also TR2.P$1; no longer TR2.P$2
Routing:
- net N$10: track 8.08 -> 21.9 mm, vias 0 -> 1
- net N$11: track 21.1 -> 12.1 mm, vias 1 -> 0
- net N$7: track 7.21 -> 11.7 mm
- net N$1: track 5.66 -> 10.1 mm
- net N$4: track 21.6 -> 17.3 mm
- net N$16: track 20.7 -> 16.5 mm
- net N$13: track 13.8 -> 16.0 mm
- added copper zone on layer 1, net GND
- added copper zone on layer 16, net GND
Other:
- outline, holes or cut-outs redrawn
- board text added: "L1"
