File: zmpt101b - 3phase din.sch (EAGLE design)
At the start: 3 parts

Commit message: 1st version
Parts:
- added D1, D2, D3: DIODE_DO-219-AB(SOD123F), Diode:DIODE_DO-219-AB(SOD123F)
- added R1, R10, R11, R12, R2, R3, R4, R5, R6, R7, R8, R9: (no value), rcl:R-EU_R1206
- added U$1, U$2: 5MMBLOCK_X9, 5mm terminal block:5MMBLOCK_X9
Connections:
- new net N$1: R3.1, U$1.P$1
- new net N$10: R5.2, TR2.A1
- new net N$11: R8.2, TR2.E1
- new net N$12: U$1.P$2
- new net N$13: R11.1, U$1.P$5
- new net N$14: R10.1, R11.2
- new net N$15: R10.2, R9.1
- new net N$16: R9.2, TR3.A1
- new net N$17: R12.2, TR3.E1
- new net N$18: U$1.P$4
- new net N$19: U$1.P$6
- new net N$2: R2.1, R3.2
- new net N$20: U$1.P$7
- new net N$21: U$1.P$8
- new net N$22: D1.C, TR1.A2, U$2.P$9
- new net N$23: D1.A, TR1.E2, U$2.P$8
- new net N$24: D2.C, TR2.A2, U$2.P$6
- new net N$25: D2.A, TR2.E2, U$2.P$5
- new net N$26: D3.C, TR3.A2, U$2.P$3
- new net N$27: D3.A, TR3.E2, U$2.P$2
- new net N$3: R1.1, R2.2
- new net N$4: R1.2, TR1.A1
- new net N$5: R4.2, TR1.E1
- new net N$6: R12.1, R4.1, R8.1, U$1.P$9
- new net N$7: R7.1, U$1.P$3
- new net N$8: R6.1, R7.2
- new net N$9: R5.1, R6.2

Commit message: commit v0.1 for prototyping
Parts:
- R1, R11, R12, R2, R3, R4, R5, R6, R7, R8, R9: value (none) -> 51k
- R10: value (none) -> 15k
Connections:
- new net GND: U$2.P$1
- net N$10: now also R8.2; no longer R5.2
- net N$11: now also R5.2; no longer R8.2
- net N$24: now also TR2.E2; no longer TR2.A2
- net N$25: now also TR2.A2; no longer TR2.E2
Changed lines of the file:
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@@
 <setting verticaltext="up"/>
 </settings>
-<grid distance="0.1" unitdist="inch" unit="inch" style="lines" multiple="1" display="no" altdistance="0.05" altunitdist="inch" altunit="inch"/>
+<grid distance="0.1" unitdist="inch" unit="inch" style="lines" multiple="1" display="no" altdistance="0.01" altunitdist="inch" altunit="inch"/>
 <layers>
 <layer number="1" name="Top" color="4" fill="1" visible="no" active="no"/>
@@
 <part name="TR2" library="ZMPT101B" deviceset="ZMPT101B" device="" package3d_urn="urn:adsk.eagle:package:14702/1"/>
 <part name="TR3" library="ZMPT101B" deviceset="ZMPT101B" device="" package3d_urn="urn:adsk.eagle:package:14702/1"/>
-<part name="R1" library="rcl" library_urn="urn:adsk.eagle:library:334" deviceset="R-EU_" device="R1206" package3d_urn="urn:adsk.eagle:package:23540/2"/>
-<part name="R2" library="rcl" library_urn="urn:adsk.eagle:library:334" deviceset="R-EU_" device="R1206" package3d_urn="urn:adsk.eagle:package:23540/2"/>
-<part name="R3" library="rcl" library_urn="urn:adsk.eagle:library:334" deviceset="R-EU_" device="R1206" package3d_urn="urn:adsk.eagle:package:23540/2"/>
-<part name="R4" library="rcl" library_urn="urn:adsk.eagle:library:334" deviceset="R-EU_" device="R1206" package3d_urn="urn:adsk.eagle:package:23540/2"/>
-<part name="R5" library="rcl" library_urn="urn:adsk.eagle:library:334" deviceset="R-EU_" device="R1206" package3d_urn="urn:adsk.eagle:package:23540/2"/>
-<part name="R6" library="rcl" library_urn="urn:adsk.eagle:library:334" deviceset="R-EU_" device="R1206" package3d_urn="urn:adsk.eagle:package:23540/2"/>
-<part name="R7" library="rcl" library_urn="urn:adsk.eagle:library:334" deviceset="R-EU_" device="R1206" package3d_urn="urn:adsk.eagle:package:23540/2"/>
-<part name="R8" library="rcl" library_urn="urn:adsk.eagle:library:334" deviceset="R-EU_" device="R1206" package3d_urn="urn:adsk.eagle:package:23540/2"/>
-<part name="R9" library="rcl" library_urn="urn:adsk.eagle:library:334" deviceset="R-EU_" device="R1206" package3d_urn="urn:adsk.eagle:package:23540/2"/>
-<part name="R10" library="rcl" library_urn="urn:adsk.eagle:library:334" deviceset="R-EU_" device="R1206" package3d_urn="urn:adsk.eagle:package:23540/2"/>
-<part name="R11" library="rcl" library_urn="urn:adsk.eagle:library:334" deviceset="R-EU_" device="R1206" package3d_urn="urn:adsk.eagle:package:23540/2"/>
-<part name="R12" library="rcl" library_urn="urn:adsk.eagle:library:334" deviceset="R-EU_" device="R1206" package3d_urn="urn:adsk.eagle:package:23540/2"/>
+<part name="R1" library="rcl" library_urn="urn:adsk.eagle:library:334" deviceset="R-EU_" device="R1206" package3d_urn="urn:adsk.eagle:package:23540/2" value="51k"/>
+<part name="R2" library="rcl" library_urn="urn:adsk.eagle:library:334" deviceset="R-EU_" device="R1206" package3d_urn="urn:adsk.eagle:package:23540/2" value="51k"/>
+<part name="R3" library="rcl" library_urn="urn:adsk.eagle:library:334" deviceset="R-EU_" device="R1206" package3d_urn="urn:adsk.eagle:package:23540/2" value="51k"/>
+<part name="R4" library="rcl" library_urn="urn:adsk.eagle:library:334" deviceset="R-EU_" device="R1206" package3d_urn="urn:adsk.eagle:package:23540/2" value="51k"/>
+<part name="R5" library="rcl" library_urn="urn:adsk.eagle:library:334" deviceset="R-EU_" device="R1206" package3d_urn="urn:adsk.eagle:package:23540/2" value="51k"/>
+<part name="R6" library="rcl" library_urn="urn:adsk.eagle:library:334" deviceset="R-EU_" device="R1206" package3d_urn="urn:adsk.eagle:package:23540/2" value="51k"/>
+<part name="R7" library="rcl" library_urn="urn:adsk.eagle:library:334" deviceset="R-EU_" device="R1206" package3d_urn="urn:adsk.eagle:package:23540/2" value="51k"/>
+<part name="R8" library="rcl" library_urn="urn:adsk.eagle:library:334" deviceset="R-EU_" device="R1206" package3d_urn="urn:adsk.eagle:package:23540/2" value="51k"/>
+<part name="R9" library="rcl" library_urn="urn:adsk.eagle:library:334" deviceset="R-EU_" device="R1206" package3d_urn="urn:adsk.eagle:package:23540/2" value="51k"/>
+<part name="R10" library="rcl" library_urn="urn:adsk.eagle:library:334" deviceset="R-EU_" device="R1206" package3d_urn="urn:adsk.eagle:package:23540/2" value="15k"/>
+<part name="R11" library="rcl" library_urn="urn:adsk.eagle:library:334" deviceset="R-EU_" device="R1206" package3d_urn="urn:adsk.eagle:package:23540/2" value="51k"/>
+<part name="R12" library="rcl" library_urn="urn:adsk.eagle:library:334" deviceset="R-EU_" device="R1206" package3d_urn="urn:adsk.eagle:package:23540/2" value="51k"/>
 <part name="U$1" library="5mm terminal block" deviceset="5MMBLOCK_X9" device=""/>
 <part name="U$2" library="5mm terminal block" deviceset="5MMBLOCK_X9" device=""/>
@@
 <part name="D2" library="Diode" library_urn="urn:adsk.eagle:library:16378169" deviceset="DIODE" device="DO-219-AB(SOD123F)" package3d_urn="urn:adsk.eagle:package:9427153/2" technology="_"/>
 <part name="D3" library="Diode" library_urn="urn:adsk.eagle:library:16378169" deviceset="DIODE" device="DO-219-AB(SOD123F)" package3d_urn="urn:adsk.eagle:package:9427153/2" technology="_"/>
+<part name="SUPPLY1" library="supply2" library_urn="urn:adsk.eagle:library:372" deviceset="GND" device=""/>
 </parts>
 <sheets>
@@
 <instance part="D3" gate="G$1" x="43.18" y="25.4" smashed="yes" rot="R90">
 <attribute name="NAME" x="38.1" y="25.4" size="1.778" layer="95" rot="R90" align="center"/>
+</instance>
+<instance part="SUPPLY1" gate="GND" x="55.88" y="10.16" smashed="yes">
+<attribute name="VALUE" x="53.975" y="6.985" size="1.778" layer="96"/>
 </instance>
 </instances>
@@
 </segment>
 </net>
-<net name="N$10" class="0">
-<segment>
-<pinref part="R5" gate="G$1" pin="2"/>
-<pinref part="TR2" gate="G$1" pin="A1"/>
-<wire x1="17.78" y1="43.18" x2="22.86" y2="43.18" width="0.1524" layer="91"/>
-</segment>
-</net>
-<net name="N$11" class="0">
-<segment>
-<pinref part="TR2" gate="G$1" pin="E1"/>
-<pinref part="R8" gate="G$1" pin="2"/>
-<wire x1="22.86" y1="35.56" x2="17.78" y2="35.56" width="0.1524" layer="91"/>
-</segment>
-</net>
 <net name="N$13" class="0">
 <segment>
@@
 <net name="N$24" class="0">
 <segment>
-<pinref part="TR2" gate="G$1" pin="A2"/>
 <pinref part="U$2" gate="G$1" pin="P$6"/>
-<wire x1="33.02" y1="43.18" x2="43.18" y2="43.18" width="0.1524" layer="91"/>
 <pinref part="D2" gate="G$1" pin="C"/>
 <wire x1="45.72" y1="43.18" x2="58.42" y2="43.18" width="0.1524" layer="91"/>
@@
 <junction x="43.18" y="45.72"/>
 <junction x="45.72" y="43.18"/>
+<pinref part="TR2" gate="G$1" pin="E2"/>
+<wire x1="43.18" y1="45.72" x2="33.02" y2="35.56" width="0.1524" layer="91"/>
 </segment>
 </net>
 <net name="N$25" class="0">
 <segment>
-<pinref part="TR2" gate="G$1" pin="E2"/>
 <pinref part="U$2" gate="G$1" pin="P$5"/>
-<wire x1="33.02" y1="35.56" x2="33.02" y2="38.1" width="0.1524" layer="91"/>
-<wire x1="33.02" y1="38.1" x2="45.72" y2="38.1" width="0.1524" layer="91"/>
 <pinref part="D2" gate="G$1" pin="A"/>
 <wire x1="45.72" y1="38.1" x2="58.42" y2="38.1" width="0.1524" layer="91"/>
 <wire x1="43.18" y1="35.56" x2="45.72" y2="35.56" width="0.1524" layer="91"/>
 <wire x1="45.72" y1="35.56" x2="45.72" y2="38.1" width="0.1524" layer="91"/>
-<junction x="45.72" y="38.1"/>
+<pinref part="TR2" gate="G$1" pin="A2"/>
+<wire x1="33.02" y1="43.18" x2="43.18" y2="35.56" width="0.1524" layer="91"/>
+<junction x="43.18" y="35.56"/>
 </segment>
 </net>
@@
 </segment>
 </net>
+<net name="GND" class="0">
+<segment>
+<pinref part="U$2" gate="G$1" pin="P$1"/>
+<wire x1="58.42" y1="17.78" x2="55.88" y2="17.78" width="0.1524" layer="91"/>
+<wire x1="55.88" y1="17.78" x2="55.88" y2="12.7" width="0.1524" layer="91"/>
+<pinref part="SUPPLY1" gate="GND" pin="GND"/>
+</segment>
+</net>
+<net name="N$10" class="0">
+<segment>
+<pinref part="R8" gate="G$1" pin="2"/>
+<pinref part="TR2" gate="G$1" pin="A1"/>
+<wire x1="17.78" y1="35.56" x2="22.86" y2="43.18" width="0.1524" layer="91"/>
+</segment>
+</net>
+<net name="N$11" class="0">
+<segment>
+<pinref part="R5" gate="G$1" pin="2"/>
+<pinref part="TR2" gate="G$1" pin="E1"/>
+<wire x1="17.78" y1="43.18" x2="22.86" y2="35.56" width="0.1524" layer="91"/>
+</segment>
+</net>
